File: Optical Encoder Schematic and Board/Optical Encoder 10-17-16.brd (EAGLE design)
At the start: 58.1 x 43.2 mm, 30 parts, among them U1 ATMEGA328P, Y1 16MHz

Commit message: updated boards
Parts:
- moved R3 1.27 mm to (3.81, 14.0)
- moved JP1 1.27 mm to (3.81, 30.5)
- moved POWER 1.27 mm to (2.54, 10.2)
- moved J4 0.92 mm to (3.05, 5.84)
Routing:
- net N$4: track 37.6 -> 12.9 mm, vias 2 -> 0
- net D5: track 31.5 -> 54.8 mm, vias 1 -> 0
- net D3: track 53.0 -> 30.7 mm, vias 0 -> 1
- net D4: track 30.4 -> 51.7 mm
- net VCC: track 187.6 -> 201.2 mm, vias 1 -> 2
- net GND: track 216.5 -> 226.5 mm, vias 4 -> 5
- net RXI: track 45.4 -> 36.0 mm, vias 0 -> 1
- net N$5: track 13.8 -> 21.1 mm, vias 0 -> 2
- net N$6: track 14.9 -> 21.0 mm, vias 2 -> 0
- net RESET: track 43.8 -> 49.3 mm, vias 3 -> 2
- net TXO: track 22.0 -> 25.4 mm
- net AREF: track 18.8 -> 16.8 mm
- net SCK: track 20.0 -> 18.3 mm
- net SDA: track 30.9 -> 29.9 mm
- net N$1: track 9.46 -> 8.81 mm
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