File: Optical Encoder Schematic and Board/Optical Encoder.sch (EAGLE design)
At the start: 30 parts, among them U1 ATMEGA328P, Y1 16MHz

Commit message: Updated Optical encoder board with latest changes. Added 2 status LEDs to ICSP board.
Parts:
- removed R7: 4.7k, SparkFun-Resistors:RESISTOR1206
- added R11: 150, SparkFun-Passives:RESISTOR0603-RES
- R10, R6, R8, R9: device SparkFun-Resistors:RESISTOR1206 -> SparkFun-Passives:RESISTOR0603-RES
- R3: value 150 -> 4.7k; device SparkFun-Resistors:RESISTOR1206 -> SparkFun-Passives:RESISTOR0603-RES
Connections:
- net D3: now also R8.2; no longer R9.2
- net D4: now also R9.2; no longer R8.2
- net N$20: now also R9.1; no longer R8.1
- net N$7: now also R8.1; no longer R9.1
- net N$9: now also R11.1; no longer R3.1
- net SCL: now also R6.1; no longer R7.1
- net SDA: now also R3.1; no longer R6.1
- net VCC: now also R11.2; no longer R7.2
Other:
- moved on the sheet: R3, R6, R8, R9
