File: 10 Pin ICSP Board/ICSP board.sch (EAGLE design)
At the start: 23 parts, among them U1 ATMEGA328P, U2 M5205 5v, X1 Power In, Y1 16MHz

Commit message: Updates to final board Changed power connector as discussed. Rotated some components for slightly better trace routing. Added labels to connectors and board date/version. Ready for fab.
Parts:
- removed JP2: I2C, SparkFun-Connectors:M02PTH
- removed X1: Power In, con-weidmueller-sl35:180G-2
- added POWER: 87758-0216, con-molex:87758-0216
- JP1: value FTDI Basic -> FTDI
- renumbered U$1 to ICSP
Connections:
- net D10: now also ICSP.5
- net GND: now also POWER-2.S; no longer X1.2
- net RESET: no longer ICSP.5
- net SCL: no longer JP2.2
- net SDA: no longer JP2.1
- net VIN: now also POWER-1.S; no longer X1.1
Changed lines of the file:
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@@
 <?xml version="1.0" encoding="utf-8"?>
 <!DOCTYPE eagle SYSTEM "eagle.dtd">
-<eagle version="7.7.0">
+<eagle version="7.1.0">
 <drawing>
 <settings>
@@
 </classes>
 <parts>
-<part name="JP1" library="SparkFun-Connectors" deviceset="M06" device="SIP" value="FTDI Basic"/>
+<part name="JP1" library="SparkFun-Connectors" deviceset="M06" device="SIP" value="FTDI"/>
 <part name="U1" library="SparkFun-DigitalIC" deviceset="ATMEGA328_SMT" device="" value="ATMEGA328P"/>
 <part name="SUPPLY1" library="SparkFun-Aesthetics" deviceset="VCC" device=""/>
@@
 <part name="GND13" library="SparkFun-Aesthetics" deviceset="GND" device=""/>
 <part name="S1" library="SparkFun-Electromechanical" deviceset="SWITCH-MOMENTARY-2" device="SMD" value="Reset"/>
-<part name="JP2" library="SparkFun-Connectors" deviceset="M02" device="PTH" value="I2C"/>
-<part name="X1" library="con-weidmueller-sl35" deviceset="180G-2" device="" value="Power In"/>
 <part name="D3" library="SparkFun-LED" deviceset="LED-GREEN" device="0603" value="RX"/>
-<part name="U$1" library="SparkFun-Connectors" deviceset="AVR_SPI_PROG" device=""/>
+<part name="ICSP" library="SparkFun-Connectors" deviceset="AVR_SPI_PROG" device=""/>
 <part name="GND17" library="SparkFun-Aesthetics" deviceset="GND" device=""/>
 <part name="SUPPLY5" library="SparkFun-Aesthetics" deviceset="VCC" device=""/>
+<part name="POWER" library="con-molex" deviceset="87758-0216" device=""/>
 </parts>
 <sheets>
@@
 <instance part="GND13" gate="1" x="-68.58" y="-10.16"/>
 <instance part="S1" gate="G$1" x="55.88" y="60.96" rot="R90"/>
-<instance part="JP2" gate="G$1" x="-93.98" y="20.32" rot="R180"/>
-<instance part="X1" gate="G$1" x="-71.12" y="-27.94"/>
 <instance part="D3" gate="G$1" x="-55.88" y="2.54"/>
-<instance part="U$1" gate="A" x="25.4" y="43.18"/>
+<instance part="ICSP" gate="A" x="25.4" y="43.18"/>
 <instance part="GND17" gate="1" x="43.18" y="27.94"/>
 <instance part="SUPPLY5" gate="G$1" x="40.64" y="50.8"/>
+<instance part="POWER" gate="-1" x="-25.4" y="-22.86" smashed="yes">
+<attribute name="NAME" x="-22.86" y="-23.622" size="1.524" layer="95"/>
+<attribute name="VALUE" x="-26.162" y="-21.463" size="1.778" layer="96"/>
+</instance>
+<instance part="POWER" gate="-2" x="-25.4" y="-27.94"/>
 </instances>
 <busses>
@@
 </segment>
 <segment>
-<pinref part="X1" gate="G$1" pin="2"/>
-<wire x1="-73.66" y1="-30.48" x2="-78.74" y2="-30.48" width="0.1524" layer="91"/>
-<label x="-78.74" y="-30.48" size="1.27" layer="95" rot="R180" xref="yes"/>
-</segment>
-<segment>
 <pinref part="D3" gate="G$1" pin="C"/>
 <pinref part="GND12" gate="1" pin="GND"/>
@@
 <segment>
 <pinref part="GND17" gate="1" pin="GND"/>
-<pinref part="U$1" gate="A" pin="10"/>
+<pinref part="ICSP" gate="A" pin="10"/>
 <wire x1="43.18" y1="45.72" x2="43.18" y2="43.18" width="0.1524" layer="91"/>
 <wire x1="43.18" y1="43.18" x2="43.18" y2="40.64" width="0.1524" layer="91"/>
@@
 <wire x1="35.56" y1="38.1" x2="43.18" y2="38.1" width="0.1524" layer="91"/>
 <junction x="43.18" y="38.1"/>
-<pinref part="U$1" gate="A" pin="8"/>
+<pinref part="ICSP" gate="A" pin="8"/>
 <wire x1="35.56" y1="40.64" x2="43.18" y2="40.64" width="0.1524" layer="91"/>
 <junction x="43.18" y="40.64"/>
-<pinref part="U$1" gate="A" pin="6"/>
+<pinref part="ICSP" gate="A" pin="6"/>
 <wire x1="35.56" y1="43.18" x2="43.18" y2="43.18" width="0.1524" layer="91"/>
 <junction x="43.18" y="43.18"/>
-<pinref part="U$1" gate="A" pin="4"/>
+<pinref part="ICSP" gate="A" pin="4"/>
 <wire x1="35.56" y1="45.72" x2="43.18" y2="45.72" width="0.1524" layer="91"/>
+</segment>
+<segment>
+<pinref part="POWER" gate="-2" pin="S"/>
+<wire x1="-27.94" y1="-27.94" x2="-35.56" y2="-27.94" width="0.1524" layer="91"/>
+<label x="-35.56" y="-27.94" size="1.778" layer="95" rot="R180" xref="yes"/>
 </segment>
 </net>
@@
 </segment>
 <segment>
-<pinref part="U$1" gate="A" pin="2"/>
+<pinref part="ICSP" gate="A" pin="2"/>
 <wire x1="35.56" y1="48.26" x2="40.64" y2="48.26" width="0.1524" layer="91"/>
 <wire x1="40.64" y1="48.26" x2="40.64" y2="50.8" width="0.1524" layer="91"/>
@@
 <pinref part="S1" gate="G$1" pin="2"/>
 <wire x1="55.88" y1="66.04" x2="55.88" y2="73.66" width="0.1524" layer="91"/>
-</segment>
-<segment>
-<pinref part="U$1" gate="A" pin="5"/>
-<wire x1="17.78" y1="43.18" x2="10.16" y2="43.18" width="0.1524" layer="91"/>
-<label x="10.16" y="43.18" size="1.778" layer="95" rot="R180" xref="yes"/>
 </segment>
 </net>
@@
 </segment>
 <segment>
-<pinref part="X1" gate="G$1" pin="1"/>
-<wire x1="-73.66" y1="-27.94" x2="-78.74" y2="-27.94" width="0.1524" layer="91"/>
-<label x="-78.74" y="-27.94" size="1.27" layer="95" rot="R180" xref="yes"/>
+<pinref part="POWER" gate="-1" pin="S"/>
+<wire x1="-27.94" y1="-22.86" x2="-35.56" y2="-22.86" width="0.1524" layer="91"/>
+<label x="-35.56" y="-22.86" size="1.778" layer="95" rot="R180" xref="yes"/>
 </segment>
 </net>
@@
 <label x="144.78" y="63.5" size="1.27" layer="95" xref="yes"/>
 </segment>
-<segment>
-<pinref part="JP2" gate="G$1" pin="1"/>
-<wire x1="-101.6" y1="20.32" x2="-106.68" y2="20.32" width="0.1524" layer="91"/>
-<label x="-106.68" y="20.32" size="1.27" layer="95" rot="R180" xref="yes"/>
-</segment>
 </net>
 <net name="SCL" class="0">
@@
 <label x="144.78" y="60.96" size="1.27" layer="95" xref="yes"/>
 </segment>
-<segment>
-<pinref part="JP2" gate="G$1" pin="2"/>
-<wire x1="-101.6" y1="17.78" x2="-106.68" y2="17.78" width="0.1524" layer="91"/>
-<label x="-106.68" y="17.78" size="1.27" layer="95" rot="R180" xref="yes"/>
-</segment>
 </net>
 <net name="A6" class="0">
@@
 <label x="144.78" y="22.86" size="1.27" layer="95" xref="yes"/>
 </segment>
+<segment>
+<pinref part="ICSP" gate="A" pin="5"/>
+<wire x1="17.78" y1="43.18" x2="7.62" y2="43.18" width="0.1524" layer="91"/>
+<label x="7.62" y="43.18" size="1.778" layer="95" rot="R180" xref="yes"/>
+</segment>
 </net>
 <net name="MOSI" class="0">
@@
 </segment>
 <segment>
-<pinref part="U$1" gate="A" pin="1"/>
+<pinref part="ICSP" gate="A" pin="1"/>
 <wire x1="17.78" y1="48.26" x2="10.16" y2="48.26" width="0.1524" layer="91"/>
 <label x="10.16" y="48.26" size="1.778" layer="95" rot="R180" xref="yes"/>
@@
 </segment>
 <segment>
-<pinref part="U$1" gate="A" pin="9"/>
+<pinref part="ICSP" gate="A" pin="9"/>
 <label x="7.62" y="33.02" size="1.778" layer="95" rot="R180" xref="yes"/>
 <wire x1="17.78" y1="38.1" x2="17.78" y2="33.02" width="0.1524" layer="91"/>
@@
 </segment>
 <segment>
-<pinref part="U$1" gate="A" pin="7"/>
+<pinref part="ICSP" gate="A" pin="7"/>
 <label x="7.62" y="38.1" size="1.778" layer="95" rot="R180" xref="yes"/>
 <wire x1="17.78" y1="40.64" x2="7.62" y2="40.64" width="0.1524" layer="91"/>

Commit message: Updated Optical encoder board with latest changes. Added 2 status LEDs to ICSP board.
Parts:
- added D5: ERROR, SparkFun-LED:LED-GREEN0603
- added D6: PMODE, SparkFun-LED:LED-GREEN0603
- added R6, R7: 10k, SparkFun-Passives:RESISTOR0603-RES
Connections:
- new net N$7: D5.A, R6.1
- new net N$8: D6.A, R7.1
- net D7: now also R7.2
- net D8: now also R6.2
- net GND: now also D5.C, D6.C
Changed lines of the file:
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@@
 <part name="SUPPLY5" library="SparkFun-Aesthetics" deviceset="VCC" device=""/>
 <part name="POWER" library="con-molex" deviceset="87758-0216" device=""/>
+<part name="GND14" library="SparkFun-Aesthetics" deviceset="GND" device=""/>
+<part name="GND15" library="SparkFun-Aesthetics" deviceset="GND" device=""/>
+<part name="D5" library="SparkFun-LED" deviceset="LED-GREEN" device="0603" value="ERROR"/>
+<part name="D6" library="SparkFun-LED" deviceset="LED-GREEN" device="0603" value="PMODE"/>
+<part name="R6" library="SparkFun-Passives" deviceset="RESISTOR" device="0603-RES" value="10k"/>
+<part name="R7" library="SparkFun-Passives" deviceset="RESISTOR" device="0603-RES" value="10k"/>
 </parts>
 <sheets>
@@
 </instance>
 <instance part="POWER" gate="-2" x="-25.4" y="-27.94"/>
+<instance part="GND14" gate="1" x="205.74" y="-10.16"/>
+<instance part="GND15" gate="1" x="185.42" y="-10.16"/>
+<instance part="D5" gate="G$1" x="205.74" y="7.62"/>
+<instance part="D6" gate="G$1" x="185.42" y="7.62"/>
+<instance part="R6" gate="G$1" x="205.74" y="22.86" rot="R90"/>
+<instance part="R7" gate="G$1" x="185.42" y="22.86" rot="R90"/>
 </instances>
 <busses>
@@
 <label x="-35.56" y="-27.94" size="1.778" layer="95" rot="R180" xref="yes"/>
 </segment>
+<segment>
+<pinref part="GND15" gate="1" pin="GND"/>
+<pinref part="D6" gate="G$1" pin="C"/>
+<wire x1="185.42" y1="-7.62" x2="185.42" y2="2.54" width="0.1524" layer="91"/>
+</segment>
+<segment>
+<pinref part="GND14" gate="1" pin="GND"/>
+<pinref part="D5" gate="G$1" pin="C"/>
+<wire x1="205.74" y1="-7.62" x2="205.74" y2="2.54" width="0.1524" layer="91"/>
+</segment>
 </net>
 <net name="VCC" class="0">
@@
 <label x="144.78" y="33.02" size="1.27" layer="95" xref="yes"/>
 </segment>
+<segment>
+<pinref part="R7" gate="G$1" pin="2"/>
+<wire x1="185.42" y1="27.94" x2="185.42" y2="33.02" width="0.1524" layer="91"/>
+<label x="185.42" y="33.02" size="1.778" layer="95" rot="R90" xref="yes"/>
+</segment>
 </net>
 <net name="D8" class="0">
@@
 <wire x1="137.16" y1="27.94" x2="144.78" y2="27.94" width="0.1524" layer="91"/>
 <label x="144.78" y="27.94" size="1.27" layer="95" xref="yes"/>
+</segment>
+<segment>
+<pinref part="R6" gate="G$1" pin="2"/>
+<wire x1="205.74" y1="33.02" x2="205.74" y2="27.94" width="0.1524" layer="91"/>
+<label x="205.74" y="33.02" size="1.778" layer="95" rot="R90" xref="yes"/>
 </segment>
 </net>
@@
 </segment>
 </net>
+<net name="N$7" class="0">
+<segment>
+<pinref part="D5" gate="G$1" pin="A"/>
+<pinref part="R6" gate="G$1" pin="1"/>
+<wire x1="205.74" y1="10.16" x2="205.74" y2="17.78" width="0.1524" layer="91"/>
+</segment>
+</net>
+<net name="N$8" class="0">
+<segment>
+<pinref part="R7" gate="G$1" pin="1"/>
+<pinref part="D6" gate="G$1" pin="A"/>
+<wire x1="185.42" y1="17.78" x2="185.42" y2="10.16" width="0.1524" layer="91"/>
+</segment>
+</net>
