File: RIO LEDs SMD/RoboRio LED schematic.brd (EAGLE design)
At the start: 100 x 80 mm, 50 parts

Commit message: JIT board
Parts:
- moved R13 83.9 mm to (5.08, 25.4), turned to 180 degrees
- moved D13 80.4 mm to (1.27, 27.9), turned to 90 degrees
- moved D11 80.2 mm to (1.27, 35.6)
- moved D3 80.2 mm to (1.27, 66.0)
- moved D5 80.1 mm to (1.27, 58.4)
- moved D9 80.1 mm to (1.27, 43.2)
- moved D7 80.0 mm to (1.27, 50.8)
- moved R12 79.0 mm to (10.2, 38.1), turned to 0 degrees
- moved R10 78.8 mm to (10.2, 45.7), turned to 0 degrees
- moved R4 78.8 mm to (10.2, 68.6), turned to 0 degrees
- moved R6 78.8 mm to (10.2, 61.0), turned to 0 degrees
- moved R8 78.8 mm to (10.2, 53.3), turned to 0 degrees
- moved R11 76.6 mm to (5.08, 33.0), turned to 180 degrees
- moved R9 76.4 mm to (5.08, 40.6), turned to 180 degrees
- moved R3 76.2 mm to (5.08, 63.5), turned to 180 degrees
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Routing:
- net S3: track 0.00 -> 9.79 mm
- net S: track 0.00 -> 9.79 mm
- net S9: track 0.00 -> 9.79 mm
- net S6: track 0.00 -> 9.79 mm
- net S8: track 0.00 -> 9.71 mm
- net S5: track 0.00 -> 9.71 mm
- net S2: track 0.00 -> 9.71 mm
- net S1: track 0.00 -> 9.70 mm
- net S4: track 0.00 -> 9.70 mm
- net S7: track 0.00 -> 9.70 mm
- net GND7: track 0.00 -> 4.53 mm
- net GND4: track 0.00 -> 4.53 mm
- net GND1: track 0.00 -> 4.53 mm
- net GND3: track 0.00 -> 4.44 mm
- net GND: track 0.00 -> 4.44 mm
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Other:
- board size 100 x 80 mm -> 15.2 x 80 mm
- board text added: "+"
- board text added: "G"
- board text added: "High"
- board text added: "Low"
- board text added: "S"
