File: RoboRio LED schematic.sch (EAGLE design)
At the start: 50 parts

Commit message: Trial layouts, smaller components, no need to review
Parts:
- D1, D10, D11, D12, D13, D14, D15, D16, D17, D18, D19, D2, D20, D3, D4, D5, D6, D7, D8, D9: device SparkFun-LED:LED1206 -> LilyPad-Wearables:LED1206
- R1, R10, R11, R12, R13, R14, R15, R16, R17, R18, R19, R2, R20, R3, R4, R5, R6, R7, R8, R9: device SparkFun-Passives:RESISTOR1206 -> SparkFun-Passives:RESISTOR0603-RES
Changed lines of the file:
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@@
 </classes>
 <parts>
-<part name="R1" library="SparkFun-Passives" deviceset="RESISTOR" device="1206"/>
-<part name="R2" library="SparkFun-Passives" deviceset="RESISTOR" device="1206"/>
 <part name="J1" library="SparkFun-Connectors" deviceset="M03" device="PTH"/>
-<part name="D1" library="SparkFun-LED" deviceset="LED" device="1206"/>
-<part name="D2" library="SparkFun-LED" deviceset="LED" device="1206"/>
-<part name="R3" library="SparkFun-Passives" deviceset="RESISTOR" device="1206"/>
-<part name="R4" library="SparkFun-Passives" deviceset="RESISTOR" device="1206"/>
+<part name="D1" library="LilyPad-Wearables" deviceset="LED" device="1206"/>
+<part name="D2" library="LilyPad-Wearables" deviceset="LED" device="1206"/>
+<part name="R3" library="SparkFun-Passives" deviceset="RESISTOR" device="0603-RES"/>
+<part name="R4" library="SparkFun-Passives" deviceset="RESISTOR" device="0603-RES"/>
 <part name="J2" library="SparkFun-Connectors" deviceset="M03" device="PTH"/>
-<part name="D3" library="SparkFun-LED" deviceset="LED" device="1206"/>
-<part name="D4" library="SparkFun-LED" deviceset="LED" device="1206"/>
-<part name="R5" library="SparkFun-Passives" deviceset="RESISTOR" device="1206"/>
-<part name="R6" library="SparkFun-Passives" deviceset="RESISTOR" device="1206"/>
+<part name="D3" library="LilyPad-Wearables" deviceset="LED" device="1206"/>
+<part name="D4" library="LilyPad-Wearables" deviceset="LED" device="1206"/>
+<part name="R5" library="SparkFun-Passives" deviceset="RESISTOR" device="0603-RES"/>
+<part name="R6" library="SparkFun-Passives" deviceset="RESISTOR" device="0603-RES"/>
 <part name="J3" library="SparkFun-Connectors" deviceset="M03" device="PTH"/>
-<part name="D5" library="SparkFun-LED" deviceset="LED" device="1206"/>
-<part name="D6" library="SparkFun-LED" deviceset="LED" device="1206"/>
-<part name="R7" library="SparkFun-Passives" deviceset="RESISTOR" device="1206"/>
-<part name="R8" library="SparkFun-Passives" deviceset="RESISTOR" device="1206"/>
+<part name="D5" library="LilyPad-Wearables" deviceset="LED" device="1206"/>
+<part name="D6" library="LilyPad-Wearables" deviceset="LED" device="1206"/>
+<part name="R7" library="SparkFun-Passives" deviceset="RESISTOR" device="0603-RES"/>
+<part name="R8" library="SparkFun-Passives" deviceset="RESISTOR" device="0603-RES"/>
 <part name="J4" library="SparkFun-Connectors" deviceset="M03" device="PTH"/>
-<part name="D7" library="SparkFun-LED" deviceset="LED" device="1206"/>
-<part name="D8" library="SparkFun-LED" deviceset="LED" device="1206"/>
-<part name="R9" library="SparkFun-Passives" deviceset="RESISTOR" device="1206"/>
-<part name="R10" library="SparkFun-Passives" deviceset="RESISTOR" device="1206"/>
+<part name="D7" library="LilyPad-Wearables" deviceset="LED" device="1206"/>
+<part name="D8" library="LilyPad-Wearables" deviceset="LED" device="1206"/>
+<part name="R9" library="SparkFun-Passives" deviceset="RESISTOR" device="0603-RES"/>
+<part name="R10" library="SparkFun-Passives" deviceset="RESISTOR" device="0603-RES"/>
 <part name="J5" library="SparkFun-Connectors" deviceset="M03" device="PTH"/>
-<part name="D9" library="SparkFun-LED" deviceset="LED" device="1206"/>
-<part name="D10" library="SparkFun-LED" deviceset="LED" device="1206"/>
-<part name="R11" library="SparkFun-Passives" deviceset="RESISTOR" device="1206"/>
-<part name="R12" library="SparkFun-Passives" deviceset="RESISTOR" device="1206"/>
+<part name="D9" library="LilyPad-Wearables" deviceset="LED" device="1206"/>
+<part name="D10" library="LilyPad-Wearables" deviceset="LED" device="1206"/>
+<part name="R11" library="SparkFun-Passives" deviceset="RESISTOR" device="0603-RES"/>
+<part name="R12" library="SparkFun-Passives" deviceset="RESISTOR" device="0603-RES"/>
 <part name="J6" library="SparkFun-Connectors" deviceset="M03" device="PTH"/>
-<part name="D11" library="SparkFun-LED" deviceset="LED" device="1206"/>
-<part name="D12" library="SparkFun-LED" deviceset="LED" device="1206"/>
-<part name="R13" library="SparkFun-Passives" deviceset="RESISTOR" device="1206"/>
-<part name="R14" library="SparkFun-Passives" deviceset="RESISTOR" device="1206"/>
+<part name="D11" library="LilyPad-Wearables" deviceset="LED" device="1206"/>
+<part name="D12" library="LilyPad-Wearables" deviceset="LED" device="1206"/>
+<part name="R13" library="SparkFun-Passives" deviceset="RESISTOR" device="0603-RES"/>
+<part name="R14" library="SparkFun-Passives" deviceset="RESISTOR" device="0603-RES"/>
 <part name="J7" library="SparkFun-Connectors" deviceset="M03" device="PTH"/>
-<part name="D13" library="SparkFun-LED" deviceset="LED" device="1206"/>
-<part name="D14" library="SparkFun-LED" deviceset="LED" device="1206"/>
-<part name="R15" library="SparkFun-Passives" deviceset="RESISTOR" device="1206"/>
-<part name="R16" library="SparkFun-Passives" deviceset="RESISTOR" device="1206"/>
+<part name="D13" library="LilyPad-Wearables" deviceset="LED" device="1206"/>
+<part name="D14" library="LilyPad-Wearables" deviceset="LED" device="1206"/>
+<part name="R15" library="SparkFun-Passives" deviceset="RESISTOR" device="0603-RES"/>
+<part name="R16" library="SparkFun-Passives" deviceset="RESISTOR" device="0603-RES"/>
 <part name="J8" library="SparkFun-Connectors" deviceset="M03" device="PTH"/>
-<part name="D15" library="SparkFun-LED" deviceset="LED" device="1206"/>
-<part name="D16" library="SparkFun-LED" deviceset="LED" device="1206"/>
-<part name="R17" library="SparkFun-Passives" deviceset="RESISTOR" device="1206"/>
-<part name="R18" library="SparkFun-Passives" deviceset="RESISTOR" device="1206"/>
+<part name="D15" library="LilyPad-Wearables" deviceset="LED" device="1206"/>
+<part name="D16" library="LilyPad-Wearables" deviceset="LED" device="1206"/>
+<part name="R17" library="SparkFun-Passives" deviceset="RESISTOR" device="0603-RES"/>
+<part name="R18" library="SparkFun-Passives" deviceset="RESISTOR" device="0603-RES"/>
 <part name="J9" library="SparkFun-Connectors" deviceset="M03" device="PTH"/>
-<part name="D17" library="SparkFun-LED" deviceset="LED" device="1206"/>
-<part name="D18" library="SparkFun-LED" deviceset="LED" device="1206"/>
-<part name="R19" library="SparkFun-Passives" deviceset="RESISTOR" device="1206"/>
-<part name="R20" library="SparkFun-Passives" deviceset="RESISTOR" device="1206"/>
+<part name="D17" library="LilyPad-Wearables" deviceset="LED" device="1206"/>
+<part name="D18" library="LilyPad-Wearables" deviceset="LED" device="1206"/>
+<part name="R19" library="SparkFun-Passives" deviceset="RESISTOR" device="0603-RES"/>
+<part name="R20" library="SparkFun-Passives" deviceset="RESISTOR" device="0603-RES"/>
 <part name="J10" library="SparkFun-Connectors" deviceset="M03" device="PTH"/>
-<part name="D19" library="SparkFun-LED" deviceset="LED" device="1206"/>
-<part name="D20" library="SparkFun-LED" deviceset="LED" device="1206"/>
+<part name="D19" library="LilyPad-Wearables" deviceset="LED" device="1206"/>
+<part name="D20" library="LilyPad-Wearables" deviceset="LED" device="1206"/>
+<part name="R1" library="SparkFun-Passives" deviceset="RESISTOR" device="0603-RES"/>
+<part name="R2" library="SparkFun-Passives" deviceset="RESISTOR" device="0603-RES"/>
 </parts>
 <sheets>
@@
 </plain>
 <instances>
-<instance part="R1" gate="G$1" x="27.94" y="142.24"/>
-<instance part="R2" gate="G$1" x="60.96" y="142.24"/>
 <instance part="J1" gate="J$1" x="2.54" y="142.24"/>
 <instance part="D1" gate="G$1" x="43.18" y="142.24" rot="R90"/>
@@
 <instance part="D19" gate="G$1" x="43.18" y="5.08" rot="R90"/>
 <instance part="D20" gate="G$1" x="76.2" y="5.08" rot="R90"/>
+<instance part="R1" gate="G$1" x="27.94" y="142.24"/>
+<instance part="R2" gate="G$1" x="60.96" y="142.24"/>
 </instances>
 <busses>
@@
 <wire x1="10.16" y1="144.78" x2="10.16" y2="149.86" width="0.1524" layer="91"/>
 <wire x1="10.16" y1="149.86" x2="50.8" y2="149.86" width="0.1524" layer="91"/>
-<pinref part="R2" gate="G$1" pin="1"/>
 <wire x1="48.26" y1="142.24" x2="50.8" y2="142.24" width="0.1524" layer="91"/>
 <wire x1="50.8" y1="142.24" x2="55.88" y2="142.24" width="0.1524" layer="91"/>
@@
 <pinref part="J1" gate="J$1" pin="3"/>
 <pinref part="D1" gate="G$1" pin="C"/>
+<pinref part="R2" gate="G$1" pin="1"/>
 </segment>
 </net>
@@
 <net name="N$1" class="0">
 <segment>
-<pinref part="R1" gate="G$1" pin="1"/>
 <wire x1="10.16" y1="142.24" x2="22.86" y2="142.24" width="0.1524" layer="91"/>
 <pinref part="J1" gate="J$1" pin="2"/>
+<pinref part="R1" gate="G$1" pin="1"/>
 </segment>
 </net>
 <net name="N$4" class="0">
 <segment>
-<pinref part="R2" gate="G$1" pin="2"/>
 <wire x1="66.04" y1="142.24" x2="73.66" y2="142.24" width="0.1524" layer="91"/>
 <pinref part="D2" gate="G$1" pin="A"/>
+<pinref part="R2" gate="G$1" pin="2"/>
 </segment>
 </net>
 <net name="N$2" class="0">
 <segment>
-<pinref part="R1" gate="G$1" pin="2"/>
 <wire x1="33.02" y1="142.24" x2="40.64" y2="142.24" width="0.1524" layer="91"/>
 <pinref part="D1" gate="G$1" pin="A"/>
+<pinref part="R1" gate="G$1" pin="2"/>
 </segment>
 </net>

Commit message: Added labels and removed component names from board.
Changed lines of the file:
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@@
 <?xml version="1.0" encoding="utf-8"?>
 <!DOCTYPE eagle SYSTEM "eagle.dtd">
-<eagle version="7.6.0">
+<eagle version="7.1.0">
 <drawing>
 <settings>
@@
 </plain>
 <instances>
-<instance part="J1" gate="J$1" x="2.54" y="142.24"/>
-<instance part="D1" gate="G$1" x="43.18" y="142.24" rot="R90"/>
-<instance part="D2" gate="G$1" x="76.2" y="142.24" rot="R90"/>
+<instance part="J1" gate="J$1" x="2.54" y="142.24" smashed="yes">
+<attribute name="VALUE" x="0" y="134.62" size="1.778" layer="96"/>
+</instance>
+<instance part="D1" gate="G$1" x="43.18" y="142.24" smashed="yes" rot="R90">
+<attribute name="VALUE" x="47.752" y="147.955" size="1.778" layer="96" rot="R180"/>
+</instance>
+<instance part="D2" gate="G$1" x="76.2" y="142.24" smashed="yes" rot="R90">
+<attribute name="VALUE" x="80.772" y="147.955" size="1.778" layer="96" rot="R180"/>
+</instance>
 <instance part="R3" gate="G$1" x="27.94" y="127"/>
 <instance part="R4" gate="G$1" x="60.96" y="127"/>
-<instance part="J2" gate="J$1" x="2.54" y="127"/>
-<instance part="D3" gate="G$1" x="43.18" y="127" rot="R90"/>
-<instance part="D4" gate="G$1" x="76.2" y="127" rot="R90"/>
+<instance part="J2" gate="J$1" x="2.54" y="127" smashed="yes">
+<attribute name="VALUE" x="0" y="119.38" size="1.778" layer="96"/>
+</instance>
+<instance part="D3" gate="G$1" x="43.18" y="127" smashed="yes" rot="R90">
+<attribute name="VALUE" x="47.752" y="132.715" size="1.778" layer="96" rot="R180"/>
+</instance>
+<instance part="D4" gate="G$1" x="76.2" y="127" smashed="yes" rot="R90">
+<attribute name="VALUE" x="80.772" y="132.715" size="1.778" layer="96" rot="R180"/>
+</instance>
 <instance part="R5" gate="G$1" x="27.94" y="111.76"/>
 <instance part="R6" gate="G$1" x="60.96" y="111.76"/>
-<instance part="J3" gate="J$1" x="2.54" y="111.76"/>
-<instance part="D5" gate="G$1" x="43.18" y="111.76" rot="R90"/>
-<instance part="D6" gate="G$1" x="76.2" y="111.76" rot="R90"/>
+<instance part="J3" gate="J$1" x="2.54" y="111.76" smashed="yes">
+<attribute name="VALUE" x="0" y="104.14" size="1.778" layer="96"/>
+</instance>
+<instance part="D5" gate="G$1" x="43.18" y="111.76" smashed="yes" rot="R90">
+<attribute name="VALUE" x="47.752" y="117.475" size="1.778" layer="96" rot="R180"/>
+</instance>
+<instance part="D6" gate="G$1" x="76.2" y="111.76" smashed="yes" rot="R90">
+<attribute name="VALUE" x="80.772" y="117.475" size="1.778" layer="96" rot="R180"/>
+</instance>
 <instance part="R7" gate="G$1" x="27.94" y="96.52"/>
 <instance part="R8" gate="G$1" x="60.96" y="96.52"/>
-<instance part="J4" gate="J$1" x="2.54" y="96.52"/>
-<instance part="D7" gate="G$1" x="43.18" y="96.52" rot="R90"/>
-<instance part="D8" gate="G$1" x="76.2" y="96.52" rot="R90"/>
+<instance part="J4" gate="J$1" x="2.54" y="96.52" smashed="yes">
+<attribute name="VALUE" x="0" y="88.9" size="1.778" layer="96"/>
+</instance>
+<instance part="D7" gate="G$1" x="43.18" y="96.52" smashed="yes" rot="R90">
+<attribute name="VALUE" x="47.752" y="102.235" size="1.778" layer="96" rot="R180"/>
+</instance>
+<instance part="D8" gate="G$1" x="76.2" y="96.52" smashed="yes" rot="R90">
+<attribute name="VALUE" x="80.772" y="102.235" size="1.778" layer="96" rot="R180"/>
+</instance>
 <instance part="R9" gate="G$1" x="27.94" y="81.28"/>
 <instance part="R10" gate="G$1" x="60.96" y="81.28"/>
-<instance part="J5" gate="J$1" x="2.54" y="81.28"/>
-<instance part="D9" gate="G$1" x="43.18" y="81.28" rot="R90"/>
-<instance part="D10" gate="G$1" x="76.2" y="81.28" rot="R90"/>
+<instance part="J5" gate="J$1" x="2.54" y="81.28" smashed="yes">
+<attribute name="VALUE" x="0" y="73.66" size="1.778" layer="96"/>
+</instance>
+<instance part="D9" gate="G$1" x="43.18" y="81.28" smashed="yes" rot="R90">
+<attribute name="VALUE" x="47.752" y="86.995" size="1.778" layer="96" rot="R180"/>
+</instance>
+<instance part="D10" gate="G$1" x="76.2" y="81.28" smashed="yes" rot="R90">
+<attribute name="VALUE" x="80.772" y="86.995" size="1.778" layer="96" rot="R180"/>
+</instance>
 <instance part="R11" gate="G$1" x="27.94" y="66.04"/>
 <instance part="R12" gate="G$1" x="60.96" y="66.04"/>
-<instance part="J6" gate="J$1" x="2.54" y="66.04"/>
-<instance part="D11" gate="G$1" x="43.18" y="66.04" rot="R90"/>
-<instance part="D12" gate="G$1" x="76.2" y="66.04" rot="R90"/>
+<instance part="J6" gate="J$1" x="2.54" y="66.04" smashed="yes">
+<attribute name="VALUE" x="0" y="58.42" size="1.778" layer="96"/>
+</instance>
+<instance part="D11" gate="G$1" x="43.18" y="66.04" smashed="yes" rot="R90">
+<attribute name="VALUE" x="47.752" y="71.755" size="1.778" layer="96" rot="R180"/>
+</instance>
+<instance part="D12" gate="G$1" x="76.2" y="66.04" smashed="yes" rot="R90">
+<attribute name="VALUE" x="80.772" y="71.755" size="1.778" layer="96" rot="R180"/>
+</instance>
 <instance part="R13" gate="G$1" x="27.94" y="50.8"/>
 <instance part="R14" gate="G$1" x="60.96" y="50.8"/>
-<instance part="J7" gate="J$1" x="2.54" y="50.8"/>
-<instance part="D13" gate="G$1" x="43.18" y="50.8" rot="R90"/>
-<instance part="D14" gate="G$1" x="76.2" y="50.8" rot="R90"/>
+<instance part="J7" gate="J$1" x="2.54" y="50.8" smashed="yes">
+<attribute name="VALUE" x="0" y="43.18" size="1.778" layer="96"/>
+</instance>
+<instance part="D13" gate="G$1" x="43.18" y="50.8" smashed="yes" rot="R90">
+<attribute name="VALUE" x="47.752" y="56.515" size="1.778" layer="96" rot="R180"/>
+</instance>
+<instance part="D14" gate="G$1" x="76.2" y="50.8" smashed="yes" rot="R90">
+<attribute name="VALUE" x="80.772" y="56.515" size="1.778" layer="96" rot="R180"/>
+</instance>
 <instance part="R15" gate="G$1" x="27.94" y="35.56"/>
 <instance part="R16" gate="G$1" x="60.96" y="35.56"/>
-<instance part="J8" gate="J$1" x="2.54" y="35.56"/>
-<instance part="D15" gate="G$1" x="43.18" y="35.56" rot="R90"/>
-<instance part="D16" gate="G$1" x="76.2" y="35.56" rot="R90"/>
+<instance part="J8" gate="J$1" x="2.54" y="35.56" smashed="yes">
+<attribute name="VALUE" x="0" y="27.94" size="1.778" layer="96"/>
+</instance>
+<instance part="D15" gate="G$1" x="43.18" y="35.56" smashed="yes" rot="R90">
+<attribute name="VALUE" x="47.752" y="41.275" size="1.778" layer="96" rot="R180"/>
+</instance>
+<instance part="D16" gate="G$1" x="76.2" y="35.56" smashed="yes" rot="R90">
+<attribute name="VALUE" x="80.772" y="41.275" size="1.778" layer="96" rot="R180"/>
+</instance>
 <instance part="R17" gate="G$1" x="27.94" y="20.32"/>
 <instance part="R18" gate="G$1" x="60.96" y="20.32"/>
-<instance part="J9" gate="J$1" x="2.54" y="20.32"/>
-<instance part="D17" gate="G$1" x="43.18" y="20.32" rot="R90"/>
-<instance part="D18" gate="G$1" x="76.2" y="20.32" rot="R90"/>
+<instance part="J9" gate="J$1" x="2.54" y="20.32" smashed="yes">
+<attribute name="VALUE" x="0" y="12.7" size="1.778" layer="96"/>
+</instance>
+<instance part="D17" gate="G$1" x="43.18" y="20.32" smashed="yes" rot="R90">
+<attribute name="VALUE" x="47.752" y="26.035" size="1.778" layer="96" rot="R180"/>
+</instance>
+<instance part="D18" gate="G$1" x="76.2" y="20.32" smashed="yes" rot="R90">
+<attribute name="VALUE" x="80.772" y="26.035" size="1.778" layer="96" rot="R180"/>
+</instance>
 <instance part="R19" gate="G$1" x="27.94" y="5.08"/>
 <instance part="R20" gate="G$1" x="60.96" y="5.08"/>
-<instance part="J10" gate="J$1" x="2.54" y="5.08"/>
-<instance part="D19" gate="G$1" x="43.18" y="5.08" rot="R90"/>
-<instance part="D20" gate="G$1" x="76.2" y="5.08" rot="R90"/>
+<instance part="J10" gate="J$1" x="2.54" y="5.08" smashed="yes">
+<attribute name="VALUE" x="0" y="-2.54" size="1.778" layer="96"/>
+</instance>
+<instance part="D19" gate="G$1" x="43.18" y="5.08" smashed="yes" rot="R90">
+<attribute name="VALUE" x="47.752" y="10.795" size="1.778" layer="96" rot="R180"/>
+</instance>
+<instance part="D20" gate="G$1" x="76.2" y="5.08" smashed="yes" rot="R90">
+<attribute name="VALUE" x="80.772" y="10.795" size="1.778" layer="96" rot="R180"/>
+</instance>
 <instance part="R1" gate="G$1" x="27.94" y="142.24"/>
 <instance part="R2" gate="G$1" x="60.96" y="142.24"/>
