File: RoboRio LED THOLE schematic.sch (EAGLE design)
At the start: 50 parts

Commit message: Routed the through hold board. Change LED component to indicate true component size
Parts:
- removed D1, D10, D11, D12, D13, D14, D15, D16, D17, D18, D19, D2, D20, D3, D4, D5, D6, D7, D8, D9: (no value), SparkFun-LED:LTE-302
- added LED1, LED10, LED11, LED12, LED13, LED14, LED15, LED16, LED17, LED18, LED19, LED2, LED20, LED3, LED4, LED5, LED6, LED7, LED8, LED9: (no value), led:LED3MM
Connections:
- net GND: now also LED2.C; no longer D2.C
- net GND1: now also LED4.C; no longer D4.C
- net GND2: now also LED6.C; no longer D6.C
- net GND3: now also LED8.C; no longer D8.C
- net GND4: now also LED10.C; no longer D10.C
- net GND5: now also LED12.C; no longer D12.C
- net GND6: now also LED14.C; no longer D14.C
- net GND7: now also LED16.C; no longer D16.C
- net GND8: now also LED18.C; no longer D18.C
- net GND9: now also LED20.C; no longer D20.C
- net N$11: now also LED8.A; no longer D8.A
- net N$12: now also LED7.A; no longer D7.A
- net N$14: now also LED10.A; no longer D10.A
- net N$15: now also LED9.A; no longer D9.A
- net N$17: now also LED12.A; no longer D12.A
- net N$18: now also LED11.A; no longer D11.A
- net N$2: now also LED1.A; no longer D1.A
- net N$20: now also LED14.A; no longer D14.A
- net N$21: now also LED13.A; no longer D13.A
- net N$23: now also LED16.A; no longer D16.A
- net N$24: now also LED15.A; no longer D15.A
- net N$26: now also LED18.A; no longer D18.A
- net N$27: now also LED17.A; no longer D17.A
- net N$29: now also LED20.A; no longer D20.A
- net N$30: now also LED19.A; no longer D19.A
- net N$4: now also LED2.A; no longer D2.A
- net N$5: now also LED4.A; no longer D4.A
- net N$6: now also LED3.A; no longer D3.A
- net N$8: now also LED6.A; no longer D6.A
- net N$9: now also LED5.A; no longer D5.A
- net S: now also LED1.C; no longer D1.C
- net S1: now also LED3.C; no longer D3.C
- net S2: now also LED5.C; no longer D5.C
- net S3: now also LED7.C; no longer D7.C
- net S4: now also LED9.C; no longer D9.C
- net S5: now also LED11.C; no longer D11.C
- net S6: now also LED13.C; no longer D13.C
- net S7: now also LED15.C; no longer D15.C
- net S8: now also LED17.C; no longer D17.C
- net S9: now also LED19.C; no longer D19.C
